Commit message: 修改并加入焊枪urdf

File: src/jaka_ros2/src/jaka_description/urdf/jaka_zu5.urdf (robot description, URDF)
Before this commit: robot jaka_zu5, 8 links, 7 joints
Links:
- added link tool_assembly; collision mesh filename=package://jaka_description/meshes/jaka_zu5_meshes/AssemblyS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 scale=0.001 0.001 0.001; visual mesh filename=package://jaka_description/meshes/jaka_zu5_meshes/Assembly_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 scale=0.001 0.001 0.001
Joints:
- added joint Link6_to_tool_assembly: type fixed, parent Link6, child tool_assembly, origin xyz=0 0 0 rpy=0 0 0

Commit message: 已测试基站位姿,验证焊枪urdf

File: src/jaka_ros2/src/jaka_description/urdf/jaka_zu5.urdf (robot description, URDF)
Before this commit: robot jaka_zu5, 9 links, 8 joints
Links:
- added link robot_base
- added link robot_flange
Joints:
- removed joint Link6_to_tool_assembly
- added joint Link6_to_robot_flange: type fixed, parent Link6, child robot_flange, origin xyz=0 0 0 rpy=0 0 0
- added joint link0_to_robot_base: type fixed, parent link0, child robot_base, origin xyz=0 0 0 rpy=0 0 0
- added joint robot_flange_to_tool_assembly: type fixed, parent robot_flange, child tool_assembly, origin xyz=0 0 0 rpy=0 0 0
