Commit message: 点云测试成功

File: src/jaka_ros2/src/jaka_description/urdf/jaka_zu5.urdf (robot description, URDF)
Before this commit: robot jaka_zu5, 11 links, 10 joints
Joints:
- joint joint_1: origin xyz=0 -0.00022535 0.12015 rpy=0 0 0 -> xyz=0 0 0.1194849 rpy=0 0 0
- joint joint_2: origin xyz=0 0 0 rpy=1.5708 0 0 -> xyz=0 0 0 rpy=1.5707963 0 0
- joint joint_3: origin xyz=0.43 0 0 rpy=0 0 0 -> xyz=0.43032 0 0 rpy=0 0 0
- joint joint_4: origin xyz=0.3685 -1.185E-05 -0.114 rpy=0 0 0 -> xyz=0.3685822 0 -0.1143507 rpy=0 0 0
- joint joint_5: origin xyz=0 -0.1135 0 rpy=1.5708 0 0 -> xyz=0 -0.1136025 0 rpy=1.5707963 0 0
- joint joint_6: origin xyz=0 0.107 0 rpy=-1.5708 0 0 -> xyz=0 0.1073407 0 rpy=-1.5707963 0 0
